Commit message: gets trajectory in rviz

File: src/path_planning/urdf/arm_bot.urdf (robot description, URDF)
Before this commit: robot arm_bot, 6 links, 5 joints
Links:
- added link end_effector_link
Joints:
- added joint end_effector_joint: type fixed, parent link3, child end_effector_link, origin xyz=0 8 0 rpy=0 0 0

File: src/path_planning/urdf/arm_bot.xacro (robot description, xacro)
@@ -9,4 +9,5 @@
   <xacro:property name="link_h" value="1.5" />
   <link name="world"/>
+  <link name="end_effector_link"/>
   <link name="base1">
     <visual>
@@ -146,4 +147,9 @@
       <!-- Effort is between 0 and 100 (units are %) and velocity is radians per second -->
   </joint>
+  <joint name="end_effector_joint" type="fixed">
+      <parent link="link3" />
+      <child link="end_effector_link" />
+      <origin rpy="0 0 0" xyz="0 ${l3} 0" />
+  </joint>
   <transmission name="trans_base_rotate">
       <type>transmission_interface/SimpleTransmission</type>

Commit message: fixed robot model. it's now 3dof

File: src/path_planning/urdf/arm_bot.urdf (robot description, URDF)
Before this commit: robot arm_bot, 7 links, 6 joints
Links:
- removed link link3
- link base2: geometry collision box size=1.5 1.5 7.5; visual box size=1.5 1.5 7.5
- link link1: geometry collision box size=1.5 10 1.5; visual box size=1.5 10 1.5
- link link2: geometry collision box size=1.5 12 1.5; visual box size=1.5 12 1.5
Joints:
- removed joint joint3
- joint end_effector_joint: origin xyz=0 8 0 rpy=0 0 0 -> xyz=0 12 0 rpy=0 0 0; parent link3 -> link2
- joint joint1: origin xyz=0 0 5 rpy=0 0 0 -> xyz=0 0 7.5 rpy=0 0 0
- joint joint2: origin xyz=0 2 0 rpy=0 0 0 -> xyz=0 10 0 rpy=0 0 0

File: src/path_planning/urdf/arm_bot.xacro (robot description, xacro)
@@ -1,8 +1,8 @@
 <?xml version="1.0" ?>
 <robot name="arm_bot" xmlns:xacro="http://www.ros.org/wiki/xacro">
-  <xacro:property name="l1" value="2" />
-  <xacro:property name="l2" value="10" />
-  <xacro:property name="l3" value="8" />
-  <xacro:property name="base_height" value="5" />
+  <!-- This is all in cm and radians -->
+  <xacro:property name="l1" value="10" />
+  <xacro:property name="l2" value="12" />
+  <xacro:property name="base_height" value="7.5" />
   <xacro:property name="zero" value="1e-12" />
   <xacro:property name="link_w" value="1.5" />
@@ -92,25 +92,4 @@
     </inertial>
   </link>
-  <link name="link3">
-    <visual>
-        <origin rpy="0 0 0" xyz="0 ${l3/2} 0" />
-        <geometry>
-            <box size="${link_w} ${l3} ${link_h}" />
-        </geometry>
-        <material name="blue">
-            <color rgba="0 0 .8 1" />
-        </material>
-    </visual>
-    <collision>
-        <origin rpy="0 0 0" xyz="0 ${l3/2} 0" />
-        <geometry>
-            <box size="${link_w} ${l3} ${link_h}" />
-        </geometry>
-    </collision>
-    <inertial>
-        <mass value="0.1" />
-        <inertia ixx="0.03" iyy="0.03" izz="0.03" ixy="0.0" ixz="0.0" iyz="0.0" />
-    </inertial>
-  </link>
   <joint name="fixed" type="fixed">
     <parent link="world"/>
@@ -139,16 +118,8 @@
     <!-- Effort is between 0 and 100 (units are %) and velocity is radians per second -->
   </joint>
-  <joint name="joint3" type="revolute">
+  <joint name="end_effector_joint" type="fixed">
       <parent link="link2" />
-      <child link="link3" />
+      <child link="end_effector_link" />
       <origin rpy="0 0 0" xyz="0 ${l2} 0" />
-      <axis xyz="1 0 0" />
-      <limit lower="-3.14" upper="3.14" effort="100" velocity="3"/>
-      <!-- Effort is between 0 and 100 (units are %) and velocity is radians per second -->
-  </joint>
-  <joint name="end_effector_joint" type="fixed">
-      <parent link="link3" />
-      <child link="end_effector_link" />
-      <origin rpy="0 0 0" xyz="0 ${l3} 0" />
   </joint>
   <transmission name="trans_base_rotate">
@@ -182,14 +153,4 @@
       </actuator>
   </transmission>
-  <transmission name="trans_joint3">
-      <type>transmission_interface/SimpleTransmission</type>
-      <joint name="joint3">
-          <hardwareInterface>hardware_interface/EffortJointInterface</hardwareInterface>
-      </joint>
-      <actuator name="joint3_motor">
-          <hardwareInterface>hardware_interface/EffortJointInterface</hardwareInterface>
-          <mechanicalReduction>1</mechanicalReduction>
-      </actuator>
-  </transmission>
   <gazebo>
       <plugin name="gazebo_ros_control" filename="libgazebo_ros_control.so">

Commit message: joint angles ranges and smaller next pt range

File: src/path_planning/urdf/arm_bot.urdf (robot description, URDF)
Before this commit: robot arm_bot, 6 links, 5 joints
Joints:
- joint joint1: limit lower=-3.14 upper=3.14 effort=100 velocity=3 -> lower=0 upper=3.14 effort=100 velocity=3
- joint joint2: limit lower=-3.14 upper=3.14 effort=100 velocity=3 -> lower=-1.57 upper=1.57 effort=100 velocity=3

File: src/path_planning/urdf/arm_bot.xacro (robot description, xacro)
@@ -107,5 +107,5 @@
       <origin rpy="0 0 0" xyz="0 0 ${base_height}" />
       <axis xyz="1 0 0" />
-      <limit lower="-3.14" upper="3.14" effort="100" velocity="3" />
+      <limit lower="0" upper="3.14" effort="100" velocity="3" />
       <!-- Effort is between 0 and 100 (units are %) and velocity is radians per second -->
   </joint>
@@ -115,5 +115,5 @@
     <origin rpy="0 0 0" xyz="0 ${l1} 0" />
     <axis xyz="1 0 0" />
-    <limit lower="-3.14" upper="3.14" effort="100" velocity="3"/>
+    <limit lower="-1.57" upper="1.57" effort="100" velocity="3"/>
     <!-- Effort is between 0 and 100 (units are %) and velocity is radians per second -->
   </joint>
